Commit message: testing ssh key

File: ur_configuration/urdf/ur10e_wgripper.urdf.xacro (robot description, xacro)
@@ -17,5 +17,5 @@
     <parent link="world" />
     <child link = "base_link" />
-    <origin xyz="0.0 0.0 0.0" rpy="0.0 0.0 0.0" />
+    <origin xyz="0.0 0.0 0.0" rpy="0 0 0" />
   </joint>
 </robot>
